File: board/board.kicad_pcb (KiCad board)
At the start: 2 copper layers, 21 x 13 mm, 1 part

Commit message: added silkscreen and jlc
Parts:
- added C1: 10uF, Capacitor_SMD:C_0603_1608Metric, F.Cu at (155.2, 100.8)
- added C2: 10uF, Capacitor_SMD:C_0603_1608Metric, F.Cu at (149.6, 99.8)
- added J1: 003_power, on_edge:on_edge_2x05_host, F.Cu at (161.0, 96.5)
- added J2: 003_power, on_edge:on_edge_2x05_device, F.Cu at (140.0, 96.5)
- added R1: 0R, Resistor_SMD:R_0402_1005Metric, F.Cu at (149.4, 101.8)
- added TP1: TestPoint, TestPoint:TestPoint_Pad_2.0x2.0mm, F.Cu at (146.8, 100.8)
- added U1: XC6220B331MR, Package_TO_SOT_SMD:SOT-23-5, F.Cu at (152.4, 100.5)
- moved LOGO1 4.35 mm to (149.3, 94.7)
Routing:
- net GND: track 0.00 -> 29.9 mm, vias 0 -> 2
- net /ldo/In: track 0.00 -> 21.3 mm, vias 0 -> 1
- net /ldo/3.3v: track 0.00 -> 19.1 mm, vias 0 -> 1
- net Net-(J1-GND-Pad5): track 0.00 -> 19.0 mm
- net Net-(J1-2.5V): track 0.00 -> 18.1 mm
- net Net-(J1-GND-Pad4): track 0.00 -> 17.9 mm
- net Net-(J1-1.8V): track 0.00 -> 17.5 mm
- net Net-(J1-GND-Pad2): track 0.00 -> 17.0 mm
- net Net-(J1-GND-Pad3): track 0.00 -> 16.7 mm
- net Net-(J1-1.2V): track 0.00 -> 16.2 mm
- net /ldo/En: track 0.00 -> 5.72 mm
Other:
- outline, holes or cut-outs redrawn
- board text added: "osf.100"
- board text added: "osf.b144.v1.0"
