File: board/board.kicad_sch (KiCad schematic)
At the start: 4 parts, among them J1 003_power, J2 003_power

Commit message: V1.0
Parts:
- removed TP1: TestPoint, TestPoint:TestPoint_Pad_2.0x2.0mm, symbol Connector:TestPoint
Other:
- sheet ldo ports: added none; removed En
