File: board/ldo.kicad_sch (KiCad schematic)
At the start: 4 parts, among them U1 XC6220B331MR

Commit message: V1.0
Parts:
- removed R1: 0R, Resistor_SMD:R_0402_1005Metric, symbol Device:R_Small
- removed U1: XC6220B331MR, Package_TO_SOT_SMD:SOT-23-5, symbol Regulator_Linear:XC6220B331MR
- added U5: XC6206PxxxMR, Package_TO_SOT_SMD:SOT-23-3, symbol Regulator_Linear:XC6206PxxxMR
- C1, C2: lcsc (none) -> C19702
Connections:
- net 3.3v: now also U5.2 (VO)
- net GND: now also U5.1 (GND)
- net In: now also U5.3 (VI)
